Commit message: mesh add

File: ros_workspace/src/tf2_basic/urdf/03_wheel_joint.urdf (robot description, URDF)
Before this commit: robot visual, 16 links, 15 joints
Links:
- link left_gripper: geometry visual mesh filename=package://tf2_basic/meshes/l_finger.dae
- link left_tip: geometry visual mesh filename=package://tf2_basic/meshes/l_finger_tip.dae
- link right_gripper: geometry visual mesh filename=package://tf2_basic/meshes/l_finger.dae
- link right_tip: geometry visual mesh filename=package://tf2_basic/meshes/l_finger_tip.dae
